File: gimbal_PCB.kicad_pcb (KiCad board)
At the start: 4 copper layers, 56.8 x 48.2 mm, 65 parts, among them J2 USB_B_Mini, J5 XT60PW-M, U1 STM32F446RETx, U2 SN65HVD230, U3 TPS54302, U4 ME6211C33M5, U5 USBLC6-2SC6, Y1 16MHz

Commit message: Komplementace a finalni upravy
Parts:
- removed +, -: MountingHole_Pad, MountingHole:MountingHole_2.2mm_M2_DIN965_Pad
- added CANH: Conn_01x01_Pin, Moje_soucastky:Test_point, F.Cu at (80.3, 79.1)
- added CANL: Conn_01x01_Pin, Moje_soucastky:Test_point, F.Cu at (85.6, 80.0)
- added J8: XT30PW-M, XT30PW-M:AMASS_XT30PW-M, F.Cu at (32.7, 84.8)
- added J9: Conn_01x01_Socket, Moje_soucastky:ODrive_PAD, F.Cu at (47.1, 87.3)
- added SCL: Conn_01x01_Pin, Moje_soucastky:Test_point, F.Cu at (61.6, 98.7)
- added SDA: Conn_01x01_Pin, Moje_soucastky:Test_point, F.Cu at (65.0, 98.7)
- J5: value XT60PW-M -> Conn_01x01_Socket; footprint XT60PW-M:AMASS_XT60PW-M -> Moje_soucastky:ODrive_PAD
- moved C5 15.3 mm to (59.0, 92.8), turned to 90 degrees
- moved J5 8.77 mm to (47.2, 82.2), turned to 0 degrees
- moved H4 8.40 mm to (87.5, 110.0)
- moved C20 7.35 mm to (51.5, 95.7), turned to -90 degrees
- moved H5 7.25 mm to (32.5, 110.0)
- moved R8 7.23 mm to (59.5, 106.0), turned to 180 degrees
- moved J2 7.20 mm to (71.0, 107.0)
- moved U5 7.20 mm to (70.6, 100.5)
- moved I2C 7.12 mm to (59.5, 110.4)
- moved R9 7.04 mm to (58.7, 104.3), turned to 180 degrees
- moved R7 6.72 mm to (38.5, 110.9), turned to 90 degrees
- moved D8 6.52 mm to (85.5, 96.8)
- moved C9 6.52 mm to (85.2, 104.2)
- moved D9 6.52 mm to (85.5, 99.9)
- moved R11 6.52 mm to (83.7, 97.4)
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Connections:
- J5 pad 1: napeti_z_baterie -> GND
Routing:
- net +3.3V: track 96.1 -> 34.7 mm, vias 4 -> 9
- net Net-(U3-SW): track 35.5 -> 1.99 mm
- net +5V: track 60.6 -> 30.3 mm, vias 0 -> 9
- net GND: track 91.9 -> 69.4 mm, vias 31 -> 61
- net /NRST: track 33.5 -> 43.0 mm
- net napeti_z_baterie: track 23.5 -> 16.8 mm
- net /USB_D-: track 11.8 -> 5.44 mm
- net /USB_D+: track 11.8 -> 5.59 mm
- net /I2C3_SCL: track 29.6 -> 23.8 mm
- net /I2C3_SDA: track 24.4 -> 20.1 mm
- net Net-(J1-Pin_3): track 8.86 -> 10.6 mm
- net Net-(J1-Pin_2): track 8.77 -> 10.5 mm
- net /CAN1_TX: track 7.72 -> 9.25 mm
- net Net-(U2-Rs): track 3.16 -> 4.36 mm
- net /SWCLK: track 15.9 -> 14.9 mm
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- added copper zone on B.Cu, net +3.3V
- added copper zone on F.Cu, net +3.3V
- added copper zone on B.Cu, net +5V
- added copper zone on B.Cu, net GND
- added copper zone on F.Cu, net Net-(U3-SW)
Other:
- board size 56.8 x 48.2 mm -> 61 x 41 mm

Commit message: Komplementace a finalni upravy_V2
Parts:
- D2: footprint LED_SMD:LED_0805_2012Metric -> LED_SMD:LED_0603_1608Metric
Changed lines of the file:
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@@
 		)
 		(fp_line
-			(start -3.3 -1.5)
+			(start -3.3 -2.7)
 			(end -3.3 -3.2)
 			(stroke
@@
 		(fp_line
 			(start -3.3 3.2)
-			(end -3.3 1.5)
+			(end -3.3 2.7)
 			(stroke
 				(width 0.12)
@@
 		(fp_line
 			(start 3.3 -3.2)
-			(end 3.3 -1.5)
+			(end 3.3 -2.7)
 			(stroke
 				(width 0.12)
@@
 		)
 		(fp_line
-			(start 3.3 1.5)
+			(start 3.3 2.7)
 			(end 3.3 3.2)
 			(stroke
@@
 		(fp_line
 			(start -3.15 -3.15)
-			(end -3.15 -1.5)
+			(end -3.15 -2.7)
 			(stroke
 				(width 0.1)
@@
 		(fp_line
 			(start -3.15 3.15)
-			(end -3.15 1.5)
+			(end -3.15 2.7)
 			(stroke
 				(width 0.1)
@@
 		(fp_line
 			(start 3.15 -3.15)
-			(end 3.15 -1.5)
+			(end 3.15 -2.7)
 			(stroke
 				(width 0.1)
@@
 		(fp_line
 			(start 3.15 3.15)
-			(end 3.15 1.5)
-			(stroke
-				(width 0.1)
-				(type solid)
-			)
-			(layer "F.Fab")
-		)
-		(fp_arc
-			(start -1.91 -1.91)
-			(mid 0 -2.701148)
-			(end 1.91 -1.91)
-			(stroke
-				(width 0.1)
-				(type solid)
-			)
-			(layer "F.Fab")
-		)
-		(fp_arc
-			(start 1.91 1.91)
-			(mid 0 2.701148)
-			(end -1.91 1.91)
+			(end 3.15 2.7)
 			(stroke
 				(width 0.1)
@@
 		)
 		(pad "1" smd rect
-			(at -2.75 0)
-			(size 1.5 2.4)
+			(at -2.325 0)
+			(size 2.35 5.1)
 			(layers "F.Cu" "F.Mask" "F.Paste")
 			(net 10 "Net-(U3-SW)")
@@
 		)
 		(pad "2" smd rect
-			(at 2.75 0)
-			(size 1.5 2.4)
+			(at 2.325 0)
+			(size 2.35 5.1)
 			(layers "F.Cu" "F.Mask" "F.Paste")
 			(net 8 "+5V")
@@
 		)
 	)
-	(footprint "LED_SMD:LED_0805_2012Metric"
+	(footprint "LED_SMD:LED_0603_1608Metric"
 		(layer "F.Cu")
 		(at 43.275 105.725)
-		(descr "LED SMD 0805 (2012 Metric), square (rectangular) end terminal, IPC-7351 nominal, (Body size source: https://docs.google.com/spreadsheets/d/1BsfQQcO9C6DZCsRaXUlFlo91Tg2WpOkGARC1WS5S8t0/edit?usp=sharing), generated with kicad-footprint-generator")
+		(descr "LED SMD 0603 (1608 Metric), square (rectangular) end terminal, IPC-7351 nominal, (Body size source: http://www.tortai-tech.com/upload/download/2011102023233369053.pdf), generated with kicad-footprint-generator")
 		(tags "LED")
 		(property "Reference" "D2"
-			(at -0.05 1.925 0)
+			(at -0.175 1.575 0)
 			(layer "F.SilkS")
 			(effects
@@
 		)
 		(property "Value" "LED"
-			(at 0 1.65 0)
+			(at 0 1.43 0)
 			(layer "F.Fab")
 			(hide yes)
@@
 		(attr smd)
 		(fp_line
-			(start -1.685 -0.96)
-			(end -1.685 0.96)
+			(start -1.485 -0.735)
+			(end -1.485 0.735)
 			(stroke
 				(width 0.12)
@@
 		)
 		(fp_line
-			(start -1.685 0.96)
-			(end 1 0.96)
+			(start -1.485 0.735)
+			(end 0.8 0.735)
 			(stroke
 				(width 0.12)
@@
 		)
 		(fp_line
-			(start 1 -0.96)
-			(end -1.685 -0.96)
+			(start 0.8 -0.735)
+			(end -1.485 -0.735)
 			(stroke
 				(width 0.12)
@@
 		)
 		(fp_rect
-			(start -1.68 -0.95)
-			(end 1.68 0.95)
+			(start -1.48 -0.73)
+			(end 1.48 0.73)
 			(stroke
 				(width 0.05)
@@
 		)
 		(fp_line
-			(start -1 -0.3)
-			(end -1 0.6)
+			(start -0.8 -0.1)
+			(end -0.8 0.4)
 			(stroke
 				(width 0.1)
@@
 		)
 		(fp_line
-			(start -1 0.6)
-			(end 1 0.6)
+			(start -0.8 0.4)
+			(end 0.8 0.4)
 			(stroke
 				(width 0.1)
@@
 		)
 		(fp_line
-			(start -0.7 -0.6)
-			(end -1 -0.3)
+			(start -0.5 -0.4)
+			(end -0.8 -0.1)
 			(stroke
 				(width 0.1)
@@
 		)
 		(fp_line
-			(start 1 -0.6)
-			(end -0.7 -0.6)
+			(start 0.8 -0.4)
+			(end -0.5 -0.4)
 			(stroke
 				(width 0.1)
@@
 		)
 		(fp_line
-			(start 1 0.6)
-			(end 1 -0.6)
+			(start 0.8 0.4)
+			(end 0.8 -0.4)
 			(stroke
 				(width 0.1)
@@
 			(effects
 				(font
-					(size 0.5 0.5)
-					(thickness 0.08)
+					(size 0.4 0.4)
+					(thickness 0.06)
 				)
 			)
 		)
 		(pad "1" smd roundrect
-			(at -0.9375 0)
-			(size 0.975 1.4)
+			(at -0.7875 0)
+			(size 0.875 0.95)
 			(layers "F.Cu" "F.Mask" "F.Paste")
 			(roundrect_rratio 0.25)
@@
 		)
 		(pad "2" smd roundrect
-			(at 0.9375 0)
-			(size 0.975 1.4)
+			(at 0.7875 0)
+			(size 0.875 0.95)
 			(layers "F.Cu" "F.Mask" "F.Paste")
 			(roundrect_rratio 0.25)
@@
 		)
 		(embedded_fonts no)
-		(model "${KICAD9_3DMODEL_DIR}/LED_SMD.3dshapes/LED_0805_2012Metric.step"
+		(model "${KICAD9_3DMODEL_DIR}/LED_SMD.3dshapes/LED_0603_1608Metric.step"
 			(offset
 				(xyz 0 0 0)

Commit message: Komplementace a finalni upravy_V3
Parts:
- C10, C11: value 10p -> 8p
- D1, D5, D7, D8, D9: footprint Diode_SMD:D_SOD-882 -> Diode_SMD:D_SOD-323
- moved R11 1.15 mm to (83.7, 96.2)
- moved D7 0.78 mm to (55.0, 77.1)
- moved R12 0.70 mm to (83.7, 100.2), turned to 90 degrees
- moved D9 0.70 mm to (85.5, 100.6)
- moved D1 0.67 mm to (59.8, 77.1)
- moved D8 0.60 mm to (85.5, 96.2)
- moved D5 0.46 mm to (50.3, 77.1)
- moved SWD 0.43 mm to (88.2, 94.5)
- moved C9 0.33 mm to (85.5, 104.2)
- moved GPIO 0.15 mm to (49.2, 74.3)
- moved UART 0.15 mm to (59.0, 74.3)
Routing:
- net GND: track 69.4 -> 65.3 mm, vias 61 -> 64
- net +3.3V: track 34.7 -> 36.4 mm
- net /NRST: track 43.0 -> 44.3 mm
- net /SWDIO: track 20.4 -> 21.6 mm
- net /SWCLK: track 14.9 -> 15.8 mm
