File: gimbal_PCB.kicad_pcb (KiCad board)
At the start: 4 copper layers, 61 x 41 mm, 69 parts, among them J2 USB_B_Mini, J5 Conn_01x01_Socket, J8 XT30PW-M, J9 Conn_01x01_Socket, U1 STM32F446RETx, U2 SN65HVD230, U3 TPS54302, U4 ME6211C33M5, U5 USBLC6-2SC6, Y1 16MHz

Commit message: Komplementace a finalni upravy_V5
Parts:
- added C21: 1m, Capacitor_SMD:C_0805_2012Metric, F.Cu at (54.0, 90.1)
Routing:
- net GND: track 65.3 -> 60.4 mm, vias 64 -> 56
- net +5V: track 30.3 -> 31.6 mm
- net /I2C3_SCL: track 23.8 -> 24.9 mm
- net +3.3V: track 36.4 -> 37.0 mm

Commit message: Komplementace a finalni upravy_V6
Parts:
- added R16: 500m, Resistor_SMD:R_1206_3216Metric, F.Cu at (55.5, 92.7)
- C21: footprint Capacitor_SMD:C_0805_2012Metric -> Capacitor_THT:C_Radial_D8.0mm_H11.5mm_P3.50mm
- moved C18 2.19 mm to (52.4, 99.2)
- moved R14 2.19 mm to (53.2, 101.6)
- moved U4 2.19 mm to (52.4, 96.1)
- moved C20 2.19 mm to (49.8, 96.9)
- moved D3 2.19 mm to (51.5, 101.6)
- moved C14 2.05 mm to (42.6, 102.8)
- moved R6 2.05 mm to (34.9, 110.8)
- moved C15 2.05 mm to (42.6, 100.7)
- moved D6 2.05 mm to (35.6, 94.0)
- moved R4 2.05 mm to (38.4, 103.2)
- moved R5 2.05 mm to (40.5, 111.5)
- moved C16 2.05 mm to (35.9, 99.3)
- moved C19 2.05 mm to (38.1, 110.8)
- moved L1 2.05 mm to (44.7, 95.6)
- moved R7 2.05 mm to (36.5, 110.8)
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Connections:
- C21 pad 1: +5V -> Net-(C21-Pad1)
Routing:
- net Net-(C21-Pad1): track 0.00 -> 2.26 mm
- net /SWCLK: track 15.8 -> 14.0 mm
- net /SWDIO: track 22.0 -> 20.3 mm
- net +3.3V: track 37.0 -> 35.3 mm, vias 9 -> 11
- net +5V: track 31.6 -> 32.9 mm
- net Net-(U2-Rs): track 4.36 -> 3.30 mm
- net /USB_D+: track 5.59 -> 4.71 mm
- net /CAN1_TX: track 9.25 -> 8.47 mm
- net /CAN1_RX: track 15.1 -> 14.4 mm
- net /NRST: track 44.1 -> 43.4 mm
- net Net-(D5-K): track 19.3 -> 19.8 mm
- net /USART_TX: track 13.8 -> 14.3 mm
- net /USART_RX: track 15.4 -> 15.9 mm
- net GND: track 60.4 -> 59.9 mm, vias 56 -> 58
