File: gimbal_PCB.kicad_sch (KiCad schematic)
At the start: 65 parts, among them J1 Conn_01x04_Socket, J2 USB_B_Mini, J3 Conn_01x04_Socket, J4 Conn_01x03_Pin, J5 XT60PW-M, J6 Conn_01x02_Pin, J7 Conn_01x06_Socket, U1 STM32F446RETx, U2 SN65HVD230, U3 TPS54302, U4 ME6211C33M5, U5 USBLC6-2SC6, Y1 16MHz

Commit message: Komplementace a finalni upravy
Parts:
- removed D6: SMBJ28A, SMBJ28A:DIOM5436X244N, symbol SMBJ28A:SMBJ28A
- removed H1, H2: MountingHole_Pad, MountingHole:MountingHole_2.2mm_M2_DIN965_Pad, symbol Mechanical:MountingHole_Pad
- removed J5: XT60PW-M, XT60PW-M:AMASS_XT60PW-M, symbol XT60PW-M:XT60PW-M
- added D10: SMBJ28A, SMBJ28A:DIOM5436X244N, symbol SMBJ28A:SMBJ28A
- added J10, J11, J12, J13: Conn_01x01_Pin, Moje_soucastky:Test_point, symbol Connector:Conn_01x01_Pin
- added J5, J9: Conn_01x01_Socket, Moje_soucastky:ODrive_PAD, symbol Connector:Conn_01x01_Socket
- added J8: XT30PW-M, XT30PW-M:AMASS_XT30PW-M, symbol XT30PW-M:XT30PW-M
Connections:
- net GND: now also D10.A, J5.1 (Pin_1), J8.N
- net I2C3_SCL: now also J13.1 (Pin_1)
- net I2C3_SDA: now also J12.1 (Pin_1)
- net napeti_z_baterie: now also D10.C, J8.P, J9.1 (Pin_1)
- net at D4.1 (K), J1.3 (Pin_3), R2.1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: now also J11.1 (Pin_1)
- net at D4.2 (K), J1.2 (Pin_2), R2.2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: now also J10.1 (Pin_1)
- no-connect marks 45 -> 44

Commit message: Komplementace a finalni upravy_V2
Parts:
- C10, C11: value 10p -> 8p
- D2: footprint LED_SMD:LED_0805_2012Metric -> LED_SMD:LED_0603_1608Metric
Changed lines of the file:
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@@
 			)
 		)
-		(property "Value" "10p"
+		(property "Value" "8p"
 			(at 67.564 77.47 0)
 			(effects
@@
 			)
 		)
-		(property "Footprint" "LED_SMD:LED_0805_2012Metric"
+		(property "Footprint" "LED_SMD:LED_0603_1608Metric"
 			(at 33.02 121.92 0)
 			(effects
@@
 			)
 		)
-		(property "Value" "10p"
+		(property "Value" "8p"
 			(at 85.344 77.47 0)
 			(effects

Commit message: Komplementace a finalni upravy_V3
Parts:
- D1, D5, D7, D8, D9: footprint Diode_SMD:D_SOD-882 -> Diode_SMD:D_SOD-323
Changed lines of the file:
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@@
 			)
 		)
-		(property "Footprint" "Diode_SMD:D_SOD-882"
+		(property "Footprint" "Diode_SMD:D_SOD-323"
 			(at 222.25 43.18 0)
 			(effects
@@
 			)
 		)
-		(property "Footprint" "Diode_SMD:D_SOD-882"
+		(property "Footprint" "Diode_SMD:D_SOD-323"
 			(at 226.06 87.63 0)
 			(effects
@@
 			)
 		)
-		(property "Footprint" "Diode_SMD:D_SOD-882"
+		(property "Footprint" "Diode_SMD:D_SOD-323"
 			(at 208.28 102.87 0)
 			(effects
@@
 			)
 		)
-		(property "Footprint" "Diode_SMD:D_SOD-882"
+		(property "Footprint" "Diode_SMD:D_SOD-323"
 			(at 95.25 95.25 0)
 			(effects
@@
 			)
 		)
-		(property "Footprint" "Diode_SMD:D_SOD-882"
+		(property "Footprint" "Diode_SMD:D_SOD-323"
 			(at 217.17 43.18 0)
 			(effects

Commit message: Komplementace a finalni upravy_V5
Parts:
- added C21: 1m, Capacitor_SMD:C_0805_2012Metric, symbol Device:C_Small
Connections:
- net +5V: now also C21.1
- net GND: now also C21.2
Changed lines of the file:
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@@
 	)
 	(junction
+		(at 102.87 165.1)
+		(diameter 0)
+		(color 0 0 0 0)
+	)
+	(junction
 		(at 96.52 168.91)
 		(diameter 0)
@@
 	(wire
 		(pts
+			(xy 114.3 171.45) (xy 114.3 172.72)
+		)
+		(stroke
+			(width 0)
+			(type default)
+		)
+	)
+	(wire
+		(pts
 			(xy 50.8 173.99) (xy 50.8 171.45)
 		)
@@
 	(wire
 		(pts
-			(xy 102.87 163.83) (xy 102.87 168.91)
+			(xy 102.87 163.83) (xy 102.87 165.1)
 		)
 		(stroke
@@
 	(wire
 		(pts
+			(xy 102.87 165.1) (xy 102.87 168.91)
+		)
+		(stroke
+			(width 0)
+			(type default)
+		)
+	)
+	(wire
+		(pts
 			(xy 158.75 36.83) (xy 158.75 38.1)
 		)
@@
 	(wire
 		(pts
+			(xy 114.3 165.1) (xy 102.87 165.1)
+		)
+		(stroke
+			(width 0)
+			(type default)
+		)
+	)
+	(wire
+		(pts
 			(xy 110.49 46.99) (xy 115.57 46.99)
 		)
@@
 	(wire
 		(pts
+			(xy 114.3 166.37) (xy 114.3 165.1)
+		)
+		(stroke
+			(width 0)
+			(type default)
+		)
+	)
+	(wire
+		(pts
 			(xy 41.91 173.99) (xy 41.91 172.72)
 		)
@@
 	)
 	(symbol
+		(lib_id "power:GND")
+		(at 114.3 172.72 0)
+		(unit 1)
+		(exclude_from_sim no)
+		(in_bom yes)
+		(on_board yes)
+		(dnp no)
+		(fields_autoplaced yes)
+		(property "Reference" "#PWR024"
+			(at 114.3 179.07 0)
+			(effects
+				(font
+					(size 1.27 1.27)
+				)
+				(hide yes)
+			)
+		)
+		(property "Value" "GND"
+			(at 114.3 177.8 0)
+			(effects
+				(font
+					(size 1.27 1.27)
+				)
+				(hide yes)
+			)
+		)
+		(property "Footprint" ""
+			(at 114.3 172.72 0)
+			(effects
+				(font
+					(size 1.27 1.27)
+				)
+				(hide yes)
+			)
+		)
+		(property "Datasheet" ""
+			(at 114.3 172.72 0)
+			(effects
+				(font
+					(size 1.27 1.27)
+				)
+				(hide yes)
+			)
+		)
+		(property "Description" "Power symbol creates a global label with name \"GND\" , ground"
+			(at 114.3 172.72 0)
+			(effects
+				(font
+					(size 1.27 1.27)
+				)
+				(hide yes)
+			)
+		)
+		(pin "1"
+		)
+		(instances
+			(project "gimbal_PCB"
+				(path "/a27908c3-450c-4477-bcde-3e53ed050e28"
+					(reference "#PWR024")
+					(unit 1)
+				)
+			)
+		)
+	)
+	(symbol
 		(lib_id "Device:R")
 		(at 101.6 52.07 90)
@@
 					(unit 1)
 				)
+			)
+		)
+	)
+	(symbol
+		(lib_id "Device:C_Small")
+		(at 114.3 168.91 0)
+		(unit 1)
+		(exclude_from_sim no)
+		(in_bom yes)
+		(on_board yes)
+		(dnp no)
+		(fields_autoplaced yes)
+		(property "Reference" "C21"
+			(at 116.84 167.6462 0)
+			(effects
+				(font
+					(size 1.27 1.27)
+				)
+				(justify left)
+			)
+		)
+		(property "Value" "1m"
+			(at 116.84 170.1862 0)
+			(effects
+				(font
+					(size 1.27 1.27)
+				)
+				(justify left)
+			)
+		)
+		(property "Footprint" "Capacitor_SMD:C_0805_2012Metric"
+			(at 114.3 168.91 0)
+			(effects
+				(font
+					(size 1.27 1.27)
+				)
+				(hide yes)
+			)
+		)
+		(property "Datasheet" "~"
+			(at 114.3 168.91 0)
+			(effects
+				(font
+					(size 1.27 1.27)
+				)
+				(hide yes)
+			)
+		)
+		(property "Description" "Unpolarized capacitor, small symbol"
+			(at 114.3 168.91 0)
+			(effects
+				(font
+					(size 1.27 1.27)
+				)
+				(hide yes)
+			)
+		)
+		(pin "2"
+		)
+		(pin "1"
+		)
+		(instances
+			(project ""
+				(path "/a27908c3-450c-4477-bcde-3e53ed050e28"
+					(reference "C21")
+					(unit 1)
+				)

Commit message: Komplementace a finalni upravy_V6
Parts:
- added R16: 200m, Resistor_SMD:R_1206_3216Metric, symbol Device:R_Small
- C21: footprint Capacitor_SMD:C_0805_2012Metric -> Capacitor_THT:C_Radial_D8.0mm_H11.5mm_P3.50mm
Connections:
- net +5V: now also R16.1; no longer C21.1
- new net: C21.1, R16.2
Changed lines of the file:
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@@
 	)
 	(junction
-		(at 102.87 165.1)
-		(diameter 0)
-		(color 0 0 0 0)
-	)
-	(junction
 		(at 96.52 168.91)
 		(diameter 0)
@@
 	)
 	(junction
+		(at 102.87 165.1)
+		(diameter 0)
+		(color 0 0 0 0)
+	)
+	(junction
 		(at 100.33 88.9)
 		(diameter 0)
@@
 	(wire
 		(pts
+			(xy 111.76 165.1) (xy 114.3 165.1)
+		)
+		(stroke
+			(width 0)
+			(type default)
+		)
+	)
+	(wire
+		(pts
+			(xy 102.87 165.1) (xy 102.87 168.91)
+		)
+		(stroke
+			(width 0)
+			(type default)
+		)
+	)
+	(wire
+		(pts
 			(xy 182.88 113.03) (xy 184.15 113.03)
 		)
@@
 	(wire
 		(pts
+			(xy 102.87 165.1) (xy 106.68 165.1)
+		)
+		(stroke
+			(width 0)
+			(type default)
+		)
+	)
+	(wire
+		(pts
 			(xy 198.12 82.55) (xy 198.12 83.82)
 		)
@@
 	(wire
 		(pts
-			(xy 102.87 165.1) (xy 102.87 168.91)
-		)
-		(stroke
-			(width 0)
-			(type default)
-		)
-	)
-	(wire
-		(pts
 			(xy 158.75 36.83) (xy 158.75 38.1)
 		)
@@
 	(wire
 		(pts
-			(xy 114.3 165.1) (xy 102.87 165.1)
-		)
-		(stroke
-			(width 0)
-			(type default)
-		)
-	)
-	(wire
-		(pts
 			(xy 110.49 46.99) (xy 115.57 46.99)
 		)
@@
 	)
 	(symbol
+		(lib_id "Device:R_Small")
+		(at 109.22 165.1 90)
+		(unit 1)
+		(exclude_from_sim no)
+		(in_bom yes)
+		(on_board yes)
+		(dnp no)
+		(fields_autoplaced yes)
+		(property "Reference" "R16"
+			(at 109.22 160.02 90)
+			(effects
+				(font
+					(size 1.016 1.016)
+				)
+			)
+		)
+		(property "Value" "200m"
+			(at 109.22 162.56 90)
+			(effects
+				(font
+					(size 1.27 1.27)
+				)
+			)
+		)
+		(property "Footprint" "Resistor_SMD:R_1206_3216Metric"
+			(at 109.22 165.1 0)
+			(effects
+				(font
+					(size 1.27 1.27)
+				)
+				(hide yes)
+			)
+		)
+		(property "Datasheet" "~"
+			(at 109.22 165.1 0)
+			(effects
+				(font
+					(size 1.27 1.27)
+				)
+				(hide yes)
+			)
+		)
+		(property "Description" "Resistor, small symbol"
+			(at 109.22 165.1 0)
+			(effects
+				(font
+					(size 1.27 1.27)
+				)
+				(hide yes)
+			)
+		)
+		(pin "2"
+		)
+		(pin "1"
+		)
+		(instances
+			(project ""
+				(path "/a27908c3-450c-4477-bcde-3e53ed050e28"
+					(reference "R16")
+					(unit 1)
+				)
+			)
+		)
+	)
+	(symbol
 		(lib_id "Device:C")
 		(at 114.3 33.02 0)
@@
 			)
 		)
-		(property "Footprint" "Capacitor_SMD:C_0805_2012Metric"
+		(property "Footprint" "Capacitor_THT:C_Radial_D8.0mm_H11.5mm_P3.50mm"
 			(at 114.3 168.91 0)
 			(effects
